Commit message: add RPC

File: atom_urdf/urdf/atom.urdf (robot description, URDF)
Before this commit: robot atom, 31 links, 30 joints
Links:
- removed link uidx_arm_l1_link
- removed link uidx_arm_l2_link
- removed link uidx_arm_r1_link
- removed link uidx_arm_r2_link
- added link left_elbow_pitch_link, mass 0.8548; collision box size=0.30 0.06 0.06; visual mesh filename=package://atom_urdf/meshes/left_elbow_pitch_link.STL
- added link left_shoulder_pitch_link, mass 0.4473; visual mesh filename=package://atom_urdf/meshes/left_shoulder_pitch_link.STL
- added link right_elbow_pitch_link, mass 0.8548; collision box size=0.30 0.06 0.06; visual mesh filename=package://atom_urdf/meshes/right_elbow_pitch_link.STL
- added link right_shoulder_pitch_link, mass 0.4473; visual mesh filename=package://atom_urdf/meshes/right_shoulder_pitch_link.STL
Joints:
- removed joint uidx_l_arm_joint1
- removed joint uidx_l_arm_joint2
- removed joint uidx_r_arm_joint1
- removed joint uidx_r_arm_joint2
- added joint left_elbow_pitch_joint: type revolute, parent left_shoulder_yaw_link, child left_elbow_pitch_link, origin xyz=0.00044198773719138 0 -0.130000000000198 rpy=0 0 0, axis 0 1 0, limit lower=-1.57 upper=2 effort=36 velocity=2.62
- added joint left_shoulder_pitch_joint: type revolute, parent torso_link, child left_shoulder_pitch_link, origin xyz=0 0.128 0.333 rpy=0 0 0, axis 0 1 0, limit lower=-2.97 upper=2.97 effort=56 velocity=2.62
- added joint right_elbow_pitch_joint: type revolute, parent right_shoulder_yaw_link, child right_elbow_pitch_link, origin xyz=0.000441987737191488 0 -0.130000000000198 rpy=0 0 0, axis 0 1 0, limit lower=-1.57 upper=2 effort=36 velocity=2.62
- added joint right_shoulder_pitch_joint: type revolute, parent torso_link, child right_shoulder_pitch_link, origin xyz=0 -0.128 0.333 rpy=0 0 0, axis 0 1 0, limit lower=-2.97 upper=2.97 effort=56 velocity=2.62
- joint head_pitch_joint: type fixed -> revolute
- joint head_yaw_joint: type fixed -> revolute
- joint left_elbow_roll_joint: parent uidx_arm_l2_link -> left_elbow_pitch_link; type fixed -> revolute
- joint left_shoulder_roll_joint: parent uidx_arm_l1_link -> left_shoulder_pitch_link; type fixed -> revolute
- joint left_shoulder_yaw_joint: type fixed -> revolute
- joint left_wrist_pitch_joint: type fixed -> revolute
- joint left_wrist_yaw_joint: type fixed -> revolute
- joint right_elbow_roll_joint: parent uidx_arm_r2_link -> right_elbow_pitch_link; type fixed -> revolute
- joint right_shoulder_roll_joint: parent uidx_arm_r1_link -> right_shoulder_pitch_link; type fixed -> revolute
- joint right_shoulder_yaw_joint: type fixed -> revolute
- joint right_wrist_pitch_joint: type fixed -> revolute
- joint right_wrist_yaw_joint: type fixed -> revolute
- joint torso_joint: type fixed -> revolute

File: atom_urdf/urdf/atom_gazebo.xacro (robot description, xacro)
@@ -1,699 +1,920 @@
 <?xml version="1.0"?>
-<!--
-  Atom Robot Gazebo Configuration
-  This file defines Gazebo-specific plugins and properties for the Atom robot
--->
-<robot xmlns:xacro="http://www.ros.org/wiki/xacro">
-  <xacro:macro name="atom_gazebo">
-    <!-- Gazebo Materials -->
-    <gazebo reference="pelvis">
-      <material>Gazebo/White</material>
-      <mu1>0.8</mu1>
-      <mu2>0.8</mu2>
-      <kp>1000000.0</kp>
-      <kd>1.0</kd>
-    </gazebo>
-    <gazebo reference="torso_link">
-      <material>Gazebo/White</material>
-      <mu1>0.8</mu1>
-      <mu2>0.8</mu2>
-    </gazebo>
-    <gazebo reference="head_yaw_link">
-      <material>Gazebo/Gray</material>
-    </gazebo>
-    <gazebo reference="head_pitch_link">
-      <material>Gazebo/Gray</material>
-    </gazebo>
-    <!-- Left Leg Gazebo Properties -->
-    <gazebo reference="leg_l1_link">
-      <material>Gazebo/Blue</material>
-    </gazebo>
-    <gazebo reference="leg_l2_link">
-      <material>Gazebo/Blue</material>
-    </gazebo>
-    <gazebo reference="leg_l3_link">
-      <material>Gazebo/Blue</material>
-    </gazebo>
-    <gazebo reference="leg_l4_link">
-      <material>Gazebo/Blue</material>
-    </gazebo>
-    <gazebo reference="leg_l5_link">
-      <material>Gazebo/Blue</material>
-    </gazebo>
-    <gazebo reference="leg_l6_link">
-      <material>Gazebo/Black</material>
-      <mu1>1.2</mu1>
-      <mu2>1.2</mu2>
-      <kp>1000000.0</kp>
-      <kd>1.0</kd>
-    </gazebo>
-    <!-- Right Leg Gazebo Properties (similar to left leg) -->
-    <gazebo reference="leg_r1_link">
-      <material>Gazebo/Red</material>
-    </gazebo>
-    <gazebo reference="leg_r2_link">
-      <material>Gazebo/Red</material>
-    </gazebo>
-    <gazebo reference="leg_r3_link">
-      <material>Gazebo/Red</material>
-    </gazebo>
-    <gazebo reference="leg_r4_link">
-      <material>Gazebo/Red</material>
-    </gazebo>
-    <gazebo reference="leg_r5_link">
-      <material>Gazebo/Red</material>
-    </gazebo>
-    <gazebo reference="leg_r6_link">
-      <material>Gazebo/Black</material>
-      <mu1>1.2</mu1>
-      <mu2>1.2</mu2>
-      <kp>1000000.0</kp>
-      <kd>1.0</kd>
-    </gazebo>
-    <!-- IMU Plugin -->
-    <gazebo reference="imu_link">
-      <sensor name="imu_sensor" type="imu">
-        <plugin filename="libgazebo_ros_imu_sensor.so" name="imu_plugin">
-          <ros>
-            <namespace>/atom</namespace>
-            <remapping>~/out:=imu</remapping>
-          </ros>
-          <initial_orientation_as_reference>false</initial_orientation_as_reference>
-        </plugin>
-        <always_on>true</always_on>
-        <update_rate>100</update_rate>
-        <visualize>true</visualize>
-        <imu>
-          <angular_velocity>
-            <x>
-              <noise type="gaussian">
-                <mean>0.0</mean>
-                <stddev>2e-4</stddev>
-                <bias_mean>0.0000075</bias_mean>
-                <bias_stddev>0.0000008</bias_stddev>
-              </noise>
-            </x>
-            <y>
-              <noise type="gaussian">
-                <mean>0.0</mean>
-                <stddev>2e-4</stddev>
-                <bias_mean>0.0000075</bias_mean>
-                <bias_stddev>0.0000008</bias_stddev>
-              </noise>
-            </y>
-            <z>
-              <noise type="gaussian">
-                <mean>0.0</mean>
-                <stddev>2e-4</stddev>
-                <bias_mean>0.0000075</bias_mean>
-                <bias_stddev>0.0000008</bias_stddev>
-              </noise>
-            </z>
-          </angular_velocity>
-          <linear_acceleration>
-            <x>
-              <noise type="gaussian">
-                <mean>0.0</mean>
-                <stddev>1.7e-2</stddev>
-                <bias_mean>0.1</bias_mean>
-                <bias_stddev>0.001</bias_stddev>
-              </noise>
-            </x>
-            <y>
-              <noise type="gaussian">
-                <mean>0.0</mean>
-                <stddev>1.7e-2</stddev>
-                <bias_mean>0.1</bias_mean>
-                <bias_stddev>0.001</bias_stddev>
-              </noise>
-            </y>
-            <z>
-              <noise type="gaussian">
-                <mean>0.0</mean>
-                <stddev>1.7e-2</stddev>
-                <bias_mean>0.1</bias_mean>
-                <bias_stddev>0.001</bias_stddev>
-              </noise>
-            </z>
-          </linear_acceleration>
-        </imu>
-      </sensor>
-    </gazebo>
-    <!-- ROS2 Control Plugin -->
-    <gazebo>
-      <plugin filename="libgazebo_ros2_control.so" name="gazebo_ros2_control">
-        <robot_param>robot_description</robot_param>
-        <robot_param_node>robot_state_publisher</robot_param_node>
-        <parameters>$(find atom_gazebo)/config/atom_controllers.yaml</parameters>
-      </plugin>
-    </gazebo>
-    <!-- ROS2 Control Hardware Interface -->
-    <ros2_control name="AtomHardwareInterface" type="system">
-      <hardware>
-        <plugin>gazebo_ros2_control/GazeboSystem</plugin>
-      </hardware>
-      <!-- Left leg joints -->
-      <joint name="leg_l1_joint">
-        <command_interface name="position">
-          <param name="min">-3.14</param>
-          <param name="max">3.14</param>
-        </command_interface>
-        <state_interface name="position"/>
-        <state_interface name="velocity"/>
-        <state_interface name="effort"/>
-      </joint>
-      <joint name="leg_l2_joint">
-        <command_interface name="position">
-          <param name="min">-3.14</param>
-          <param name="max">3.14</param>
-        </command_interface>
-        <state_interface name="position"/>
-        <state_interface name="velocity"/>
-        <state_interface name="effort"/>
-      </joint>
-      <joint name="leg_l3_joint">
-        <command_interface name="position">
-          <param name="min">-3.14</param>
-          <param name="max">3.14</param>
-        </command_interface>
-        <state_interface name="position"/>
-        <state_interface name="velocity"/>
-        <state_interface name="effort"/>
-      </joint>
-      <joint name="leg_l4_joint">
-        <command_interface name="position">
-          <param name="min">-3.14</param>
-          <param name="max">3.14</param>
-        </command_interface>
-        <state_interface name="position"/>
-        <state_interface name="velocity"/>
-        <state_interface name="effort"/>
-      </joint>
-      <joint name="leg_l5_joint">
-        <command_interface name="position">
-          <param name="min">-3.14</param>
-          <param name="max">3.14</param>
-        </command_interface>
-        <state_interface name="position"/>
-        <state_interface name="velocity"/>
-        <state_interface name="effort"/>
-      </joint>
-      <joint name="leg_l6_joint">
-        <command_interface name="position">
-          <param name="min">-3.14</param>
-          <param name="max">3.14</param>
-        </command_interface>
-        <state_interface name="position"/>
-        <state_interface name="velocity"/>
-        <state_interface name="effort"/>
-      </joint>
-      <!-- Right leg joints -->
-      <joint name="leg_r1_joint">
-        <command_interface name="position">
-          <param name="min">-3.14</param>
-          <param name="max">3.14</param>
-        </command_interface>
-        <state_interface name="position"/>
-        <state_interface name="velocity"/>
-        <state_interface name="effort"/>
-      </joint>
-      <joint name="leg_r2_joint">
-        <command_interface name="position">
-          <param name="min">-3.14</param>
-          <param name="max">3.14</param>
-        </command_interface>
-        <state_interface name="position"/>
-        <state_interface name="velocity"/>
-        <state_interface name="effort"/>
-      </joint>
-      <joint name="leg_r3_joint">
-        <command_interface name="position">
-          <param name="min">-3.14</param>
-          <param name="max">3.14</param>
-        </command_interface>
-        <state_interface name="position"/>
-        <state_interface name="velocity"/>
-        <state_interface name="effort"/>
-      </joint>
-      <joint name="leg_r4_joint">
-        <command_interface name="position">
-          <param name="min">-3.14</param>
-          <param name="max">3.14</param>
-        </command_interface>
-        <state_interface name="position"/>
-        <state_interface name="velocity"/>
-        <state_interface name="effort"/>
-      </joint>
-      <joint name="leg_r5_joint">
-        <command_interface name="position">
-          <param name="min">-3.14</param>
-          <param name="max">3.14</param>
-        </command_interface>
-        <state_interface name="position"/>
-        <state_interface name="velocity"/>
-        <state_interface name="effort"/>
-      </joint>
-      <joint name="leg_r6_joint">
-        <command_interface name="position">
-          <param name="min">-3.14</param>
-          <param name="max">3.14</param>
-        </command_interface>
-        <state_interface name="position"/>
-        <state_interface name="velocity"/>
-        <state_interface name="effort"/>
-      </joint>
-      <!-- Left arm joints -->
-      <joint name="uidx_l_arm_joint1">
-        <command_interface name="position">
-          <param name="min">-2.97</param>
-          <param name="max">2.97</param>
-        </command_interface>
-        <state_interface name="position"/>
-        <state_interface name="velocity"/>
-        <state_interface name="effort"/>
-      </joint>
-      <joint name="left_shoulder_roll_joint">
-        <command_interface name="position">
-          <param name="min">-0.43</param>
-          <param name="max">3.14</param>
-        </command_interface>
-        <state_interface name="position"/>
-        <state_interface name="velocity"/>
-        <state_interface name="effort"/>
-      </joint>
-      <joint name="left_shoulder_yaw_joint">
-        <command_interface name="position">
-          <param name="min">-2.97</param>
-          <param name="max">2.97</param>
-        </command_interface>
-        <state_interface name="position"/>
-        <state_interface name="velocity"/>
-        <state_interface name="effort"/>
-      </joint>
-      <joint name="uidx_l_arm_joint2">
-        <command_interface name="position">
-          <param name="min">-1.57</param>
-          <param name="max">2</param>
-        </command_interface>
-        <state_interface name="position"/>
-        <state_interface name="velocity"/>
-        <state_interface name="effort"/>
-      </joint>
-      <joint name="left_elbow_roll_joint">
-        <command_interface name="position">
-          <param name="min">-2.97</param>
-          <param name="max">2.97</param>
-        </command_interface>
-        <state_interface name="position"/>
-        <state_interface name="velocity"/>
-        <state_interface name="effort"/>
-      </joint>
-      <joint name="left_wrist_pitch_joint">
-        <command_interface name="position">
-          <param name="min">-1.57</param>
-          <param name="max">1.57</param>
-        </command_interface>
-        <state_interface name="position"/>
-        <state_interface name="velocity"/>
-        <state_interface name="effort"/>
-      </joint>
-      <joint name="left_wrist_yaw_joint">
-        <command_interface name="position">
-          <param name="min">-1.57</param>
-          <param name="max">1.57</param>
-        </command_interface>
-        <state_interface name="position"/>
-        <state_interface name="velocity"/>
-        <state_interface name="effort"/>
-      </joint>
-      <!-- Right arm joints -->
-      <joint name="uidx_r_arm_joint1">
-        <command_interface name="position">
-          <param name="min">-2.97</param>
-          <param name="max">2.97</param>
-        </command_interface>
-        <state_interface name="position"/>
-        <state_interface name="velocity"/>
-        <state_interface name="effort"/>
-      </joint>
-      <joint name="right_shoulder_roll_joint">
-        <command_interface name="position">
-          <param name="min">-3.14</param>
-          <param name="max">0.43</param>
-        </command_interface>
-        <state_interface name="position"/>
-        <state_interface name="velocity"/>
-        <state_interface name="effort"/>
-      </joint>
-      <joint name="right_shoulder_yaw_joint">
-        <command_interface name="position">
-          <param name="min">-2.97</param>
-          <param name="max">2.97</param>
-        </command_interface>
-        <state_interface name="position"/>
-        <state_interface name="velocity"/>
-        <state_interface name="effort"/>
-      </joint>
-      <joint name="uidx_r_arm_joint2">
-        <command_interface name="position">
-          <param name="min">-1.57</param>
-          <param name="max">2</param>
-        </command_interface>
-        <state_interface name="position"/>
-        <state_interface name="velocity"/>
-        <state_interface name="effort"/>
-      </joint>
-      <joint name="right_elbow_roll_joint">
-        <command_interface name="position">
-          <param name="min">-2.97</param>
-          <param name="max">2.97</param>
-        </command_interface>
-        <state_interface name="position"/>
-        <state_interface name="velocity"/>
-        <state_interface name="effort"/>
-      </joint>
-      <joint name="right_wrist_pitch_joint">
-        <command_interface name="position">
-          <param name="min">-1.57</param>
-          <param name="max">1.57</param>
-        </command_interface>
-        <state_interface name="position"/>
-        <state_interface name="velocity"/>
-        <state_interface name="effort"/>
-      </joint>
-      <joint name="right_wrist_yaw_joint">
-        <command_interface name="position">
-          <param name="min">-1.57</param>
-          <param name="max">1.57</param>
-        </command_interface>
-        <state_interface name="position"/>
-        <state_interface name="velocity"/>
-        <state_interface name="effort"/>
-      </joint>
-      <!-- Head joints -->
-      <joint name="head_yaw_joint">
-        <command_interface name="position">
-          <param name="min">-1.57</param>
-          <param name="max">1.57</param>
-        </command_interface>
-        <state_interface name="position"/>
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
File: atom_urdf/urdf/atom_lower.urdf (robot description, URDF)
Before this commit: robot atom, 32 links, 31 joints
Links:
- removed link uidx_arm_l1_link
- removed link uidx_arm_l2_link
- removed link uidx_arm_r1_link
- removed link uidx_arm_r2_link
- added link left_elbow_pitch_link, mass 0.8548; collision box size=0.30 0.06 0.06; visual mesh filename=package://atom_urdf/meshes/left_elbow_pitch_link.STL
- added link left_shoulder_pitch_link, mass 0.4473; visual mesh filename=package://atom_urdf/meshes/left_shoulder_pitch_link.STL
- added link right_elbow_pitch_link, mass 0.8548; collision box size=0.30 0.06 0.06; visual mesh filename=package://atom_urdf/meshes/right_elbow_pitch_link.STL
- added link right_shoulder_pitch_link, mass 0.4473; visual mesh filename=package://atom_urdf/meshes/right_shoulder_pitch_link.STL
Joints:
- removed joint uidx_l_arm_joint1
- removed joint uidx_l_arm_joint2
- removed joint uidx_r_arm_joint1
- removed joint uidx_r_arm_joint2
- added joint left_elbow_pitch_joint: type revolute, parent left_shoulder_yaw_link, child left_elbow_pitch_link, origin xyz=0.00044198773719138 0 -0.130000000000198 rpy=0 0 0, axis 0 1 0, limit lower=-1.57 upper=2 effort=36 velocity=2.62
- added joint left_shoulder_pitch_joint: type revolute, parent torso_link, child left_shoulder_pitch_link, origin xyz=0 0.128 0.333 rpy=0 0 0, axis 0 1 0, limit lower=-2.97 upper=2.97 effort=56 velocity=2.62
- added joint right_elbow_pitch_joint: type revolute, parent right_shoulder_yaw_link, child right_elbow_pitch_link, origin xyz=0.000441987737191488 0 -0.130000000000198 rpy=0 0 0, axis 0 1 0, limit lower=-1.57 upper=2 effort=36 velocity=2.62
- added joint right_shoulder_pitch_joint: type revolute, parent torso_link, child right_shoulder_pitch_link, origin xyz=0 -0.128 0.333 rpy=0 0 0, axis 0 1 0, limit lower=-2.97 upper=2.97 effort=56 velocity=2.62
- joint head_pitch_joint: type fixed -> revolute
- joint head_yaw_joint: type fixed -> revolute
- joint left_elbow_roll_joint: parent uidx_arm_l2_link -> left_elbow_pitch_link; type fixed -> revolute
- joint left_shoulder_roll_joint: parent uidx_arm_l1_link -> left_shoulder_pitch_link; type fixed -> revolute
- joint left_shoulder_yaw_joint: type fixed -> revolute
- joint left_wrist_pitch_joint: type fixed -> revolute
- joint left_wrist_yaw_joint: type fixed -> revolute
- joint right_elbow_roll_joint: parent uidx_arm_r2_link -> right_elbow_pitch_link; type fixed -> revolute
- joint right_shoulder_roll_joint: parent uidx_arm_r1_link -> right_shoulder_pitch_link; type fixed -> revolute
- joint right_shoulder_yaw_joint: type fixed -> revolute
- joint right_wrist_pitch_joint: type fixed -> revolute
- joint right_wrist_yaw_joint: type fixed -> revolute

File: atom_urdf/urdf/atom_wholebody.urdf (robot description, URDF)
Before this commit: robot atom, 32 links, 31 joints
Links:
- removed link uidx_arm_l1_link
- removed link uidx_arm_l2_link
- removed link uidx_arm_r1_link
- removed link uidx_arm_r2_link
- added link left_elbow_pitch_link, mass 0.8548; collision box size=0.30 0.06 0.06; visual mesh filename=package://atom_urdf/meshes/left_elbow_pitch_link.STL
- added link left_shoulder_pitch_link, mass 0.4473; visual mesh filename=package://atom_urdf/meshes/left_shoulder_pitch_link.STL
- added link right_elbow_pitch_link, mass 0.8548; collision box size=0.30 0.06 0.06; visual mesh filename=package://atom_urdf/meshes/right_elbow_pitch_link.STL
- added link right_shoulder_pitch_link, mass 0.4473; visual mesh filename=package://atom_urdf/meshes/right_shoulder_pitch_link.STL
Joints:
- removed joint uidx_l_arm_joint1
- removed joint uidx_l_arm_joint2
- removed joint uidx_r_arm_joint1
- removed joint uidx_r_arm_joint2
- added joint left_elbow_pitch_joint: type revolute, parent left_shoulder_yaw_link, child left_elbow_pitch_link, origin xyz=0.00044198773719138 0 -0.130000000000198 rpy=0 0 0, axis 0 1 0, limit lower=-1.57 upper=2 effort=36 velocity=2.62
- added joint left_shoulder_pitch_joint: type revolute, parent torso_link, child left_shoulder_pitch_link, origin xyz=0 0.128 0.333 rpy=0 0 0, axis 0 1 0, limit lower=-2.97 upper=2.97 effort=56 velocity=2.62
- added joint right_elbow_pitch_joint: type revolute, parent right_shoulder_yaw_link, child right_elbow_pitch_link, origin xyz=0.000441987737191488 0 -0.130000000000198 rpy=0 0 0, axis 0 1 0, limit lower=-1.57 upper=2 effort=36 velocity=2.62
- added joint right_shoulder_pitch_joint: type revolute, parent torso_link, child right_shoulder_pitch_link, origin xyz=0 -0.128 0.333 rpy=0 0 0, axis 0 1 0, limit lower=-2.97 upper=2.97 effort=56 velocity=2.62
- joint left_elbow_roll_joint: parent uidx_arm_l2_link -> left_elbow_pitch_link
- joint left_shoulder_roll_joint: parent uidx_arm_l1_link -> left_shoulder_pitch_link
- joint right_elbow_roll_joint: parent uidx_arm_r2_link -> right_elbow_pitch_link
- joint right_shoulder_roll_joint: parent uidx_arm_r1_link -> right_shoulder_pitch_link
